File: brd1_555_LED_Inverter.kicad_pcb (KiCad board)
At the start: 2 copper layers, 47.8 x 44.2 mm, 39 parts, among them J1 USB_C_16Pin_C167321, J3 ConnM_01x03, U2 IC_HexTriggerInverter_SN74HC0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, U3 IC_555Timer_SA555DR, U5 LDO_3V3_2A_AIC1221-33GY3TR

Commit message: Updated Version
Parts:
- moved R3 0.99 mm to (164.5, 121.2)
- moved LED3 0.99 mm to (164.6, 125.7)
- moved R6 0.87 mm to (150.2, 119.0)
- moved LED2 0.87 mm to (160.1, 123.5)
- moved LED6 0.87 mm to (150.3, 123.5)
- moved R2 0.87 mm to (160.0, 119.0)
- moved LED7 0.70 mm to (145.9, 125.9)
- moved R7 0.70 mm to (145.8, 121.3)
- moved R4 0.66 mm to (168.1, 119.5)
- moved LED4 0.66 mm to (168.2, 123.9)
- moved LED5 0.64 mm to (141.8, 124.1)
- moved R5 0.64 mm to (141.7, 119.5)
- moved G*** 0.58 mm to (155.0, 112.8)
Routing:
- net OUT: track 47.2 -> 44.6 mm
- net Net-(LED3-Pad2): track 0.00 -> 2.61 mm
- net Net-(LED7-Pad2): track 0.00 -> 2.57 mm
- net Net-(LED5-Pad2): track 0.00 -> 2.57 mm
- net Net-(LED6-Pad2): track 0.00 -> 2.47 mm
- net Net-(LED2-Pad2): track 0.00 -> 2.47 mm
- net Net-(LED4-Pad2): track 0.00 -> 2.47 mm
- net Net-(LED1-Pad2): track 0.00 -> 1.82 mm
- net Net-(R6-Pad1): track 7.69 -> 6.76 mm
- net GND: track 41.5 -> 42.4 mm
- net Net-(R5-Pad1): track 9.43 -> 10.0 mm
- net Net-(R7-Pad1): track 14.0 -> 13.4 mm
Other:
- board text added: "10k"
- board text added: "1k"
- board text added: "300"
- board text added: "50"

Commit message: Last Update - Changed width of power trace
Parts:
- moved G*** 0.58 mm to (155.5, 112.5)
Routing:
- net GND: track 42.4 -> 44.5 mm, vias 20 -> 21
- net Net-(F1-Pad1): track 9.97 -> 8.04 mm
- added copper zone on F.Cu, net Net-(F1-Pad1)

Commit message: Minor changes
Parts:
- F1: value 16V_3A -> Fuse_Trip500mA_SMD0805B020TF
- R8: value 100 -> 100R
Other:
- board text added: "Feb'25"
