File: brd1_555_LED_Inverter.kicad_sch (KiCad schematic)
At the start: 32 parts, among them J1 USB_C_16Pin_C167321, J3 ConnM_01x03, U2 IC_HexTriggerInverter_SN74HC0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, U3 IC_555Timer_SA555DR, U5 LDO_3V3_2A_AIC1221-33GY3TR

Commit message: Minor changes
Parts:
- F1: value 16V_3A -> Fuse_Trip500mA_SMD0805B020TF
- R8: value 100 -> 100R
